File: hw/vcxo.kicad_pcb (KiCad board)
At the start: 2 copper layers, 72 parts, among them J1 Conn_01x01, J2 Conn_01x01, J3 Conn_01x01, J4 Conn_01x01, J5 Conn_01x01, J6 Conn_01x01, P1 CONN_01X04, P2 BNC, P3 CONN_01X02, U1 DAC1220E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

Commit message: fixed one cap value
Parts:
- C15: value 10n -> 100n
Changed lines of the file:
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@@
       (effects (font (size 1 1) (thickness 0.15)))
     )
-    (fp_text value 10n (at 0 1.75 180) (layer F.Fab)
+    (fp_text value 100n (at 0 1.75 180) (layer F.Fab)
       (effects (font (size 1 1) (thickness 0.15)))
     )
@@
   (segment (start 145.95 103.6975) (end 143.7525 103.6975) (width 0.35) (layer F.Cu) (net 3))
   (segment (start 143.7525 103.6975) (end 142 105.45) (width 0.35) (layer F.Cu) (net 3))
-  (segment (start 165.75 92.15) (end 165.75 89.8) (width 0.45) (layer F.Cu) (net 4) (status C00000))
-  (segment (start 165.75 89.8) (end 165.85 89.7) (width 0.45) (layer F.Cu) (net 4) (status C00000))
-  (segment (start 166.75 102.3) (end 166.75 102.25) (width 0.45) (layer F.Cu) (net 4) (status C00000))
-  (segment (start 166.75 102.25) (end 164.5 100) (width 0.45) (layer F.Cu) (net 4) (status C00000))
+  (segment (start 165.75 92.15) (end 165.75 89.8) (width 0.45) (layer F.Cu) (net 4))
+  (segment (start 165.75 89.8) (end 165.85 89.7) (width 0.45) (layer F.Cu) (net 4))
+  (segment (start 166.75 102.3) (end 166.75 102.25) (width 0.45) (layer F.Cu) (net 4))
+  (segment (start 166.75 102.25) (end 164.5 100) (width 0.45) (layer F.Cu) (net 4))
   (segment (start 146.85 113.85) (end 149.2 116.2) (width 0.45) (layer F.Cu) (net 4))
   (segment (start 149.2 116.2) (end 149.2 118.2) (width 0.45) (layer F.Cu) (net 4))
   (segment (start 149.2 118.2) (end 149.95 118.95) (width 0.45) (layer F.Cu) (net 4))
-  (segment (start 149.95 118.95) (end 151.1 118.95) (width 0.45) (layer F.Cu) (net 4) (status 800000))
-  (segment (start 144.3 111.05) (end 144.3 112.05) (width 0.45) (layer F.Cu) (net 4) (status 400000))
+  (segment (start 149.95 118.95) (end 151.1 118.95) (width 0.45) (layer F.Cu) (net 4))
+  (segment (start 144.3 111.05) (end 144.3 112.05) (width 0.45) (layer F.Cu) (net 4))
   (segment (start 146.1 113.85) (end 146.85 113.85) (width 0.45) (layer F.Cu) (net 4))
   (segment (start 144.3 112.05) (end 146.1 113.85) (width 0.45) (layer F.Cu) (net 4))
-  (segment (start 146.85 113.85) (end 148.35 113.85) (width 0.45) (layer F.Cu) (net 4) (status 800000))
-  (segment (start 148.35 113.85) (end 148.95 113.25) (width 0.45) (layer F.Cu) (net 4) (status C00000))
-  (segment (start 165.95 128.65) (end 165.95 126.5) (width 0.45) (layer F.Cu) (net 4) (status C00000))
-  (segment (start 165.95 126.5) (end 166.1 126.35) (width 0.45) (layer F.Cu) (net 4) (status C00000))
+  (segment (start 146.85 113.85) (end 148.35 113.85) (width 0.45) (layer F.Cu) (net 4))
+  (segment (start 148.35 113.85) (end 148.95 113.25) (width 0.45) (layer F.Cu) (net 4))
+  (segment (start 165.95 128.65) (end 165.95 126.5) (width 0.45) (layer F.Cu) (net 4))
+  (segment (start 165.95 126.5) (end 166.1 126.35) (width 0.45) (layer F.Cu) (net 4))
   (segment (start 153.6 127.9) (end 153.6 128.4) (width 0.35) (layer F.Cu) (net 4))
   (segment (start 153.6 128.4) (end 154.3 129.1) (width 0.35) (layer F.Cu) (net 4))

Commit message: fixed some L value
Parts:
- L1: value 1u -> 150n; footprint Inductors_SMD:L_Taiyo-Yuden_NR-30xx_HandSoldering -> Inductors_SMD:L_0805_HandSoldering
Routing:
- net GND: track 64.3 -> 68.4 mm
Changed lines of the file:
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@@
     (thickness 1.6)
     (drawings 0)
-    (tracks 247)
+    (tracks 249)
     (zones 0)
     (modules 72)
@@
   )
   (setup
-    (last_trace_width 0.45)
+    (last_trace_width 0.25)
     (user_trace_width 0.3)
     (user_trace_width 0.35)
@@
     )
   )
-  (module Inductors_SMD:L_Taiyo-Yuden_NR-30xx_HandSoldering (layer F.Cu)
-    (at 171.6 124.7 90)
-    (descr "Inductor, Taiyo Yuden, NR series, Taiyo-Yuden_NR-30xx, 3.0mmx3.0mm")
-    (tags "inductor taiyo-yuden nr smd")
-    (attr smd)
-    (fp_text reference L1 (at 0 -2.5 90) (layer F.SilkS)
-      (effects (font (size 1 1) (thickness 0.15)))
-    )
-    (fp_text value 1u (at 0 3 90) (layer F.Fab)
-      (effects (font (size 1 1) (thickness 0.15)))
-    )
-    (fp_text user %R (at 0 0 90) (layer F.Fab)
-      (effects (font (size 0.7 0.7) (thickness 0.105)))
-    )
-    (fp_line (start -1.5 0) (end -1.5 -0.95) (layer F.Fab) (width 0.1))
-    (fp_line (start -1.5 -0.95) (end -0.95 -1.5) (layer F.Fab) (width 0.1))
-    (fp_line (start -0.95 -1.5) (end 0 -1.5) (layer F.Fab) (width 0.1))
-    (fp_line (start 1.5 0) (end 1.5 -0.95) (layer F.Fab) (width 0.1))
-    (fp_line (start 1.5 -0.95) (end 0.95 -1.5) (layer F.Fab) (width 0.1))
-    (fp_line (start 0.95 -1.5) (end 0 -1.5) (layer F.Fab) (width 0.1))
-    (fp_line (start 1.5 0) (end 1.5 0.95) (layer F.Fab) (width 0.1))
-    (fp_line (start 1.5 0.95) (end 0.95 1.5) (layer F.Fab) (width 0.1))
-    (fp_line (start 0.95 1.5) (end 0 1.5) (layer F.Fab) (width 0.1))
-    (fp_line (start -1.5 0) (end -1.5 0.95) (layer F.Fab) (width 0.1))
-    (fp_line (start -1.5 0.95) (end -0.95 1.5) (layer F.Fab) (width 0.1))
-    (fp_line (start -0.95 1.5) (end 0 1.5) (layer F.Fab) (width 0.1))
-    (fp_line (start -2.5 -1.6) (end 2.5 -1.6) (layer F.SilkS) (width 0.12))
-    (fp_line (start -2.5 1.6) (end 2.5 1.6) (layer F.SilkS) (width 0.12))
-    (fp_line (start -2.75 -1.8) (end -2.75 1.8) (layer F.CrtYd) (width 0.05))
-    (fp_line (start -2.75 1.8) (end 2.75 1.8) (layer F.CrtYd) (width 0.05))
-    (fp_line (start 2.75 1.8) (end 2.75 -1.8) (layer F.CrtYd) (width 0.05))
-    (fp_line (start 2.75 -1.8) (end -2.75 -1.8) (layer F.CrtYd) (width 0.05))
-    (pad 1 smd rect (at -1.6 0 90) (size 1.8 2.9) (layers F.Cu F.Paste F.Mask)
-      (net 14 "Net-(C15-Pad2)"))
-    (pad 2 smd rect (at 1.6 0 90) (size 1.8 2.9) (layers F.Cu F.Paste F.Mask)
-      (net 15 "Net-(C16-Pad1)"))
-    (model ${KISYS3DMOD}/Inductors_SMD.3dshapes/L_Taiyo-Yuden_NR-30xx.wrl
-      (at (xyz 0 0 0))
-      (scale (xyz 1 1 1))
-      (rotate (xyz 0 0 0))
-    )
-  )
   (module Inductors_SMD:L_0805_HandSoldering (layer F.Cu)
     (at 165.75 111.95 90)
@@
     )
   )
+  (module Inductors_SMD:L_0805_HandSoldering (layer F.Cu)
+    (at 171.6 124.65 90)
+    (descr "Resistor SMD 0805, hand soldering")
+    (tags "resistor 0805")
+    (attr smd)
+    (fp_text reference L1 (at 0 -2.1 90) (layer F.SilkS)
+      (effects (font (size 1 1) (thickness 0.15)))
+    )
+    (fp_text value 150n (at 0 2.1 90) (layer F.Fab)
+      (effects (font (size 1 1) (thickness 0.15)))
+    )
+    (fp_text user %R (at 0 0 90) (layer F.Fab)
+      (effects (font (size 0.5 0.5) (thickness 0.075)))
+    )
+    (fp_line (start -1 0.62) (end -1 -0.62) (layer F.Fab) (width 0.1))
+    (fp_line (start 1 0.62) (end -1 0.62) (layer F.Fab) (width 0.1))
+    (fp_line (start 1 -0.62) (end 1 0.62) (layer F.Fab) (width 0.1))
+    (fp_line (start -1 -0.62) (end 1 -0.62) (layer F.Fab) (width 0.1))
+    (fp_line (start -2.4 -1) (end 2.4 -1) (layer F.CrtYd) (width 0.05))
+    (fp_line (start -2.4 1) (end 2.4 1) (layer F.CrtYd) (width 0.05))
+    (fp_line (start -2.4 -1) (end -2.4 1) (layer F.CrtYd) (width 0.05))
+    (fp_line (start 2.4 -1) (end 2.4 1) (layer F.CrtYd) (width 0.05))
+    (fp_line (start 0.6 0.88) (end -0.6 0.88) (layer F.SilkS) (width 0.12))
+    (fp_line (start -0.6 -0.88) (end 0.6 -0.88) (layer F.SilkS) (width 0.12))
+    (pad 1 smd rect (at -1.35 0 90) (size 1.5 1.3) (layers F.Cu F.Paste F.Mask)
+      (net 14 "Net-(C15-Pad2)"))
+    (pad 2 smd rect (at 1.35 0 90) (size 1.5 1.3) (layers F.Cu F.Paste F.Mask)
+      (net 15 "Net-(C16-Pad1)"))
+    (model ${KISYS3DMOD}/Inductors_SMD.3dshapes/L_0805.wrl
+      (at (xyz 0 0 0))
+      (scale (xyz 1 1 1))
+      (rotate (xyz 0 0 0))
+    )
+  )
   (segment (start 141.6 103.15) (end 137.6 103.15) (width 0.35) (layer F.Cu) (net 1))
   (segment (start 137.6 103.15) (end 137.35 102.9) (width 0.35) (layer F.Cu) (net 1))
   (segment (start 145.95 103.0625) (end 141.6875 103.0625) (width 0.35) (layer F.Cu) (net 1))
   (segment (start 141.6875 103.0625) (end 141.6 103.15) (width 0.35) (layer F.Cu) (net 1))
+  (segment (start 173.7 124.6) (end 169.85 124.6) (width 0.25) (layer F.Cu) (net 2))
+  (segment (start 169.85 124.6) (end 169.7 124.75) (width 0.25) (layer F.Cu) (net 2))
   (segment (start 156.65 99.25) (end 156.65 98.8) (width 0.45) (layer F.Cu) (net 2))
   (segment (start 156.65 98.8) (end 156.05 98.2) (width 0.45) (layer F.Cu) (net 2))
